File: Modulus.kicad_pcb (KiCad board)
At the start: 2 copper layers, 296.2 x 63.1 mm, 234 parts, among them J1 XLR3, J2 USB_C_Receptacle_USB2.0_16P, J3 USB_A, J4 USB_A, J5 XLR3, J6 OLED_128x32, SW1 Push_Button, U1 RP2040, U2 NCP1117-1.5_SOT223, U3 W25Q128JVS, Y1 12MHz, Y2 12MHz

Commit message: wired everything, but didn't run DRC-
Parts:
- removed Control2: Keyswitch, ScottoKeebs_Hotswap:Hotswap_MX_1.00u
- removed D83: Diode, Diode_SMD:D_SMA
- -_D1, 0)D1, 1!D1, 2@D1, 3#D1, 4$D1, 5%D1, 6^D1, 7&D1, 8*D1, 9(D1, =+D1, BackspaceD1, BackspaceD2, D31, D32, D33, D34, D35, D36, D37, D38, D39, D40, D41, D42, D43, D44, D45, D46, D47, D48, D49, D50, D51, D52, D53, D54, D55, D56, D57, D58, D59, D60, D61, D62, D63, D64, D65, D66, D67, D68, D69, D70, D71, D72, D73, D74, D75, D76, D77, D78, D79, D80, D81, D82, D84, D85, D86, D87, D88, D89, `~D1: moved to B.Cu
- S60: footprint ScottoKeebs_Hotswap:Hotswap_MX_1.50u -> ScottoKeebs_Hotswap:Hotswap_MX_1.25u
- S72: footprint ScottoKeebs_Hotswap:Hotswap_MX_1.25u -> ScottoKeebs_Hotswap:Hotswap_MX_1.50u
- UP1: footprint ScottoKeebs_MX:MX_PCB_1.00u -> ScottoKeebs_Hotswap:Hotswap_MX_1.00u
- moved Right1 455.1 mm to (295.7, 183.6)
- moved PgDown1 440.2 mm to (295.7, 164.6)
- moved Down1 437.0 mm to (276.7, 183.6)
- moved PgUp1 418.5 mm to (257.6, 164.6)
- moved Left1 410.9 mm to (257.6, 183.6)
- moved Command2 391.7 mm to (219.5, 164.6)
- moved Backspace2 387.0 mm to (295.7, 88.3)
- moved Option2 384.3 mm to (238.6, 164.6)
- moved Backspace1 377.9 mm to (276.7, 88.3)
- moved \|1 358.1 mm to (291.0, 107.4)
- moved =+1 357.0 mm to (257.6, 88.3)
- moved D73 351.3 mm to (36.4, 170.3)
- moved S58 344.4 mm to (293.3, 126.5)
- moved D74 340.3 mm to (55.4, 170.3)
- moved -_1 336.7 mm to (238.6, 88.3)
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- renumbered S34 to E1, S39 to I1, S40 to O1, S41 to P1, S32 to Q1, S35 to RKey1, S36 to T1, S31 to Tab1, S38 to UKey1, S33 to W1, S37 to YKey11, S42 to [{1, S44 to \|1, S43 to ]}1
Connections:
- Down1 pad 1: COL_12 -> COL_11
- GL850G1 pad 11: unconnected-(GL850G1-DM4-Pad11) -> PORT2_USB_D-
- GL850G1 pad 12: unconnected-(GL850G1-DP4-Pad12) -> PORT2_USB_D+
- GL850G1 pad 2: PORT2_USB_D- -> unconnected-(GL850G1-DM2-Pad2)
- GL850G1 pad 3: PORT2_USB_D+ -> unconnected-(GL850G1-DP2-Pad3)
- Left1 pad 1: COL_11 -> COL_10
- PgDown1 pad 1: COL_13 -> COL_12
- PgUp1 pad 1: COL_11 -> COL_10
- Right1 pad 1: COL_13 -> COL_12
- UP1 pad 1: COL_12 -> COL_11
Routing:
- net ROW_5: track 0.00 -> 562.4 mm, vias 0 -> 1
- net ROW_4: track 0.00 -> 537.8 mm, vias 0 -> 1
- net ROW_3: track 0.00 -> 513.0 mm, vias 0 -> 1
- net ROW_2: track 0.00 -> 498.3 mm, vias 0 -> 1
- net ROW_1: track 0.00 -> 486.5 mm, vias 0 -> 1
- net ROW_6: track 0.00 -> 352.8 mm, vias 0 -> 1
- net COL_11: track 120.3 -> 281.3 mm, vias 1 -> 13
- net COL_10: track 102.4 -> 260.0 mm, vias 1 -> 13
- net COL_9: track 82.6 -> 224.3 mm, vias 1 -> 11
- net COL_12: track 140.4 -> 281.9 mm, vias 1 -> 13
- net COL_8: track 65.2 -> 205.2 mm, vias 1 -> 11
- net ROW_0: track 339.7 -> 467.4 mm, vias 0 -> 1
- net COL_7: track 62.9 -> 186.1 mm, vias 1 -> 11
- net OLED_SDA: track 246.0 -> 123.8 mm
- net COL_6: track 43.4 -> 161.6 mm, vias 1 -> 11
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- added copper zone on F.Cu, net TEST
Other:
- board size 296.2 x 63.1 mm -> 295.6 x 183 mm

Commit message: rewired some stuff, added some new stuff
Parts:
- C1, C10, C11, C12, C17, C2, C22, C23, C24, C25, C26, C27, C3, C4, C5, C6, C7, C8, C9: footprint Capacitor_SMD:C_0402_1005Metric -> Capacitor_SMD:C_1206_3216Metric
- C13, C14: footprint Capacitor_SMD:C_0201_0603Metric -> Capacitor_SMD:C_1206_3216Metric
- C15, C16, C20, C21: footprint Capacitor_SMD:C_0201_0603Metric -> Capacitor_SMD:C_0805_2012Metric
- R1, R10, R2: footprint PCM_Resistor_SMD_AKL:R_0201_0603Metric -> Resistor_SMD:R_0805_2012Metric; moved to B.Cu
- R11, R13, R3, R4: footprint PCM_Resistor_SMD_AKL:R_0402_1005Metric -> Resistor_SMD:R_0402_1005Metric
- R12, R15: footprint PCM_Resistor_SMD_AKL:R_1206_3216Metric -> Resistor_SMD:R_1206_3216Metric; moved to B.Cu
- R16, R17, R7: footprint PCM_Resistor_SMD_AKL:R_1206_3216Metric -> Resistor_SMD:R_1206_3216Metric
- R8: footprint PCM_Resistor_SMD_AKL:R_0402_1005Metric -> Resistor_SMD:R_0805_2012Metric; moved to B.Cu
- R9: footprint PCM_Resistor_SMD_AKL:R_0402_1005Metric -> Resistor_SMD:R_0805_2012Metric
- U2: moved to B.Cu
- moved C22 79.9 mm to (88.1, 25.6), turned to 0 degrees
- moved C25 77.9 mm to (88.1, 35.7), turned to 0 degrees
- moved U2 77.3 mm to (190.5, 31.2)
- moved C26 76.9 mm to (88.1, 39.0), turned to 0 degrees
- moved C27 76.0 mm to (88.1, 42.4), turned to 0 degrees
- moved C23 69.0 mm to (88.1, 29.0)
- moved R11 54.9 mm to (106.9, 25.6)
- moved C4 52.7 mm to (76.8, 32.4), turned to 0 degrees
- moved C5 52.7 mm to (76.8, 35.7), turned to 0 degrees
- moved C3 51.8 mm to (76.8, 29.0), turned to 0 degrees
- moved D91 51.6 mm to (107.3, 29.6), turned to 0 degrees
- moved C6 51.4 mm to (76.8, 39.0), turned to 0 degrees
- moved C2 51.1 mm to (76.8, 25.6), turned to 0 degrees
- moved C1 50.7 mm to (76.8, 22.3), turned to 0 degrees
- moved C7 50.3 mm to (76.8, 42.4), turned to 0 degrees
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Routing:
- net ROW_0: track 467.4 -> 291.9 mm, vias 1 -> 0
- net ROW_1: track 486.5 -> 311.9 mm, vias 1 -> 0
- net ROW_2: track 498.3 -> 324.4 mm, vias 1 -> 0
- net ROW_3: track 513.0 -> 340.1 mm, vias 1 -> 0
- net ROW_4: track 537.8 -> 365.4 mm, vias 1 -> 0
- net ROW_6: track 352.8 -> 181.6 mm, vias 1 -> 0
- net ROW_5: track 562.4 -> 398.5 mm, vias 1 -> 0
- net COL_14: track 192.5 -> 31.8 mm, vias 3 -> 2
- net +3V3: track 219.1 -> 69.0 mm, vias 0 -> 1
- net COL_13: track 240.8 -> 99.0 mm, vias 9 -> 8
- net COL_12: track 281.9 -> 156.0 mm, vias 13 -> 12
- net COL_11: track 281.3 -> 155.6 mm, vias 13 -> 12
- net OLED_SCL: track 125.8 -> 16.5 mm, vias 2 -> 1
- net OLED_SDA: track 123.8 -> 15.4 mm, vias 2 -> 1
- net COL_10: track 260.0 -> 153.5 mm, vias 13 -> 12
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- added copper zone on B.Cu, net TEST

Commit message: rerouted AGAIn
Parts:
- C22: moved to B.Cu
- moved J6 247.8 mm to (267.2, 41.7)
- moved R16 240.0 mm to (265.5, 46.0), turned to 90 degrees
- moved R17 237.3 mm to (262.7, 46.0), turned to 90 degrees
- moved D91 161.7 mm to (268.7, 40.6), turned to 180 degrees
- moved C1 128.7 mm to (202.5, 50.4), turned to -90 degrees
- moved C2 124.8 mm to (199.1, 50.4), turned to -90 degrees
- moved C3 120.9 mm to (195.8, 50.4), turned to -90 degrees
- moved C9 118.2 mm to (199.1, 44.7), turned to 90 degrees
- moved C4 117.0 mm to (192.4, 50.4), turned to -90 degrees
- moved C17 116.5 mm to (202.5, 44.7), turned to 90 degrees
- moved C8 115.5 mm to (195.8, 44.7), turned to 90 degrees
- moved C5 113.2 mm to (189.1, 50.4), turned to -90 degrees
- moved C6 109.5 mm to (185.7, 50.4), turned to -90 degrees
- moved C7 105.8 mm to (182.4, 50.4), turned to -90 degrees
- moved C27 104.3 mm to (192.4, 44.7), turned to -90 degrees
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Routing:
- net +3V3: track 69.0 -> 351.6 mm, vias 1 -> 17
- net ROW_4: track 365.4 -> 551.2 mm, vias 0 -> 25
- net ROW_3: track 340.1 -> 505.7 mm, vias 0 -> 27
- net ROW_2: track 324.4 -> 485.6 mm, vias 0 -> 27
- net ROW_1: track 311.9 -> 471.7 mm, vias 0 -> 27
- net ROW_0: track 291.9 -> 446.4 mm, vias 0 -> 29
- net ROW_6: track 181.6 -> 335.4 mm, vias 0 -> 1
- net ROW_5: track 398.5 -> 548.2 mm, vias 0 -> 7
- net COL_14: track 31.8 -> 167.8 mm, vias 2 -> 1
- net COL_13: track 99.0 -> 219.0 mm, vias 8 -> 1
- net Net-(D91-A): track 2.31 -> 114.5 mm
- net OLED_SDA: track 15.4 -> 125.1 mm, vias 1 -> 0
- net COL_11: track 155.6 -> 264.3 mm, vias 12 -> 1
- net OLED_SCL: track 16.5 -> 122.1 mm, vias 1 -> 0
- net COL_0: track 129.7 -> 234.1 mm, vias 0 -> 1
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