File: Modulus.kicad_pcb (KiCad board)
At the start: 2 copper layers, 295.6 x 183 mm, 232 parts, among them J1 XLR3, J2 USB_C_Receptacle_USB2.0_16P, J3 USB_A, J4 USB_A, J5 XLR3, J6 OLED_128x32, P1 Keyswitch, Q1 Keyswitch, SW1 Push_Button, T1 Keyswitch, U1 RP2040, U2 NCP1117-1.5_SOT223, U3 W25Q128JVS, Y1 12MHz, Y2 12MHz

Commit message: finished the case and PCB designls doing BOM now
Parts:
- Caps Lock: renamed from S45
- Caps Lock: renamed from D91
- Comma/Open Angle Bracket: renamed from S68
- Down Arrow: renamed from Down1
- F10/Macro 1: renamed from F10
- F11/Macro 2: renamed from F11
- F12/Macro 3: renamed from F12
- F2/Increase Volume: renamed from F2
- F3/Decrease Volume: renamed from F3
- F4/Print Screen: renamed from F4
- F5/Next Track: renamed from F5
- F6/Play/Pause Media: renamed from F6
- F7/Previous Track: renamed from F7
- Five/Percent Sign: renamed from 5%1
- Four/Dollar Symbol: renamed from 4$1
- Grave Accent/Tilde: renamed from `~1
- Left Arrow: renamed from Left1
- Left Shift: renamed from S59
- Left Shift: renamed from S60
- Left Square/Curly Bracket: renamed from [{1
- Macro 4: renamed from Del1
- Nine/Open Bracket: renamed from 9(1
- One/Exclaimation Mark: renamed from 1!1
- Page Down: renamed from PgDown1
- Page Up: renamed from PgUp1
- Period/Close Angle Bracket: renamed from S69
- Quotation Mark/Apostrophe: renamed from S56
- Right Arrow: renamed from Right1
- Right Shift: renamed from S71
- Right Shift: renamed from S72
- Right Square/Curly Bracket: renamed from ]}1
- Slash/Question Mark: renamed from S70
- Two/At Sign: renamed from 2@1
- Up Arrow: renamed from UP1
- Zero/Close Bracket: renamed from 0)1
- renumbered S46 to A, Option1 to Alternate/Option, Option2 to Alternate/Option, S65 to B, \|1 to Backslash/Pipe, Backspace2 to Backspace, Backspace1 to Backspace, S63 to C, Control1 to Control, S48 to D, Del2 to Delete, E1 to E, 8*1 to Eight/Asterisk, S58 to Enter, S57 to Enter, =+1 to Equals/Plus, Esc1 to Esc, S49 to F, F1 to F1/Mute, F8 to F8/Spotlight, F9 to F9/Screenshot, Fn1 to Function, S50 to G, S51 to H, I1 to I, S52 to J, S53 to K, S54 to L, S67 to M, -_1 to Minus/Underscore, S66 to N, O1 to O, P1 to P, Q1 to Q, RKey1 to R, S47 to S, S55 to Semi-colon/Colon, 7&1 to Seven/Ampersand, 6^1 to Six/Caret, Space1 to Space, Space3 to Space, Space2 to Space, Space4 to Space, Command1 to Super/Command, Command2 to Super/Command, T1 to T, Tab1 to Tab, 3#1 to Three/Hashtag, UKey1 to U, S64 to V, W1 to W, S62 to X, YKey11 to Y, S61 to Z
Routing:
- net +3V3: track 351.6 -> 336.1 mm, vias 17 -> 18
- net Net-(GL850G1-~{OVCUR1}): track 1.83 -> 11.6 mm, vias 0 -> 1
Other:
- outline, holes or cut-outs redrawn
- board text added: "A modulur keyboard"
- board text added: "CSn VBUS"
- board text added: "D+ D-"
- board text added: "GND SC"
- board text added: "Made by @advaitconty"
- board text added: "Modulus"
- board text added: "Port 1"
- board text added: "Port 2"
- board text added: "Powered by an RP2040"
- board text added: "RX"
- board text added: "TX"
