File: Modulus.kicad_pcb (KiCad board)
At the start: 2 copper layers, 295.6 x 183 mm, 229 parts, among them J1 XLR3, J2 USB_C_Receptacle_USB2.0_16P, J3 USB_A, J4 USB_A, J5 XLR3, J6 OLED_128x32, P1 Keyswitch, Q1 Keyswitch, T1 Keyswitch, U1 RP2040, U3 W25Q128JVS, U4 NCP1117-3.3_SOT223, Y1 12MHz, Y2 12MHz

Commit message: Moved everything to the back
Parts:
- added Reset: Push_Button, Button_Switch_THT:SW_PUSH_6mm, F.Cu at (25.6, 36.2)
- C1, C10, C11, C12, C13, C14, C15, C16, C17, C2, C20, C21, C23, C24, C25, C26, C27, C3, C4, C5, C6, C7, C8, C9, GL850G1, J2, J3, J4, R1, R11, R14, R16, R17, R3, R4, R5, R6, R7, R9, U1, U3, U4, Y1, Y2: moved to B.Cu
- Caps Lock: footprint Green_LED:0603 -> LED_THT:LED_D5.0mm
- moved R11 106.9 mm to (269.3, 33.9)
- moved R7 103.0 mm to (31.5, 40.0), turned to 0 degrees
- moved J3 78.0 mm to (200.5, 24.1), turned to 0 degrees
- moved J4 78.0 mm to (122.5, 24.1), turned to 0 degrees
- moved R6 77.8 mm to (31.4, 42.8)
- moved C16 30.6 mm to (122.6, 46.0), turned to 0 degrees
- moved R13 28.7 mm to (182.3, 35.7)
- moved R5 25.8 mm to (127.9, 40.5)
- moved C15 24.3 mm to (126.9, 51.1), turned to 0 degrees
- moved R12 23.4 mm to (176.6, 36.0), turned to 180 degrees
- moved C22 21.6 mm to (152.9, 22.0), turned to 0 degrees
- moved U3 20.4 mm to (150.3, 47.1), turned to 0 degrees
- moved C1 20.1 mm to (182.4, 50.4)
- moved C14 20.1 mm to (202.5, 44.7)
- moved C17 20.1 mm to (182.4, 44.7)
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Routing:
- net ROW_6: track 335.4 -> 548.3 mm, vias 1 -> 2
- net QSPI_SS: track 50.5 -> 222.2 mm, vias 2 -> 4
- net CAPS_LOCK_LED: track 15.7 -> 150.1 mm, vias 0 -> 2
- net Net-(D91-A): track 114.5 -> 2.59 mm
- net +3V3: track 353.7 -> 441.3 mm, vias 19 -> 15
- net COL_7: track 198.0 -> 152.3 mm, vias 1 -> 2
- net COL_14: track 167.8 -> 210.7 mm, vias 1 -> 4
- net COL_13: track 219.0 -> 260.3 mm, vias 1 -> 4
- net COL_12: track 259.7 -> 293.9 mm, vias 1 -> 4
- net XLR_TX: track 20.1 -> 54.0 mm, vias 1 -> 3
- net TEST: track 12.0 -> 42.4 mm, vias 0 -> 2
- net COL_6: track 170.2 -> 145.1 mm, vias 1 -> 2
- net QSPI_SD0: track 35.2 -> 12.4 mm
- net QSPI_SD3: track 41.9 -> 19.9 mm
- net +1V1: track 66.3 -> 45.3 mm, vias 5 -> 2
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Other:
- board text added: "- may be"
- board text added: "Authorised typists only"
- board text added: "LDO"
- board text added: "RP2040"
- board text added: "WARNING"
- board text added: "hot"
- board text added: "may be hot"
- board text removed: "LDO - may be hot"
