File: Modulus.kicad_sch (KiCad schematic)
At the start: 232 parts, among them J1 XLR3, J2 USB_C_Receptacle_USB2.0_16P, J3 USB_A, J4 USB_A, J5 XLR3, J6 OLED_128x32, P1 Keyswitch, Q1 Keyswitch, SW1 Push_Button, T1 Keyswitch, U1 RP2040, U2 NCP1117-1.5_SOT223, U3 W25Q128JVS, Y1 12MHz, Y2 12MHz

Commit message: rewired some stuff, added some new stuff
Parts:
- C1, C10, C11, C12, C17, C2, C22, C23, C24, C25, C26, C27, C3, C4, C5, C6, C7, C8, C9: footprint Capacitor_SMD:C_0402_1005Metric -> Capacitor_SMD:C_1206_3216Metric
- C13, C14: footprint Capacitor_SMD:C_0201_0603Metric -> Capacitor_SMD:C_1206_3216Metric
- C15, C16, C20, C21: footprint Capacitor_SMD:C_0201_0603Metric -> Capacitor_SMD:C_0805_2012Metric
- R1, R10, R2: footprint PCM_Resistor_SMD_AKL:R_0201_0603Metric -> Resistor_SMD:R_0805_2012Metric
- R11, R13, R3, R4: footprint PCM_Resistor_SMD_AKL:R_0402_1005Metric -> Resistor_SMD:R_0402_1005Metric
- R12, R15, R16, R17, R7: footprint PCM_Resistor_SMD_AKL:R_1206_3216Metric -> Resistor_SMD:R_1206_3216Metric
- R8, R9: footprint PCM_Resistor_SMD_AKL:R_0402_1005Metric -> Resistor_SMD:R_0805_2012Metric
Other:
- moved on the sheet: C22, R15
Changed lines of the file:
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@@
 	)
 	(junction
-		(at 450.85 182.88)
+		(at 450.85 181.61)
 		(diameter 0)
 		(color 0 0 0 0)
@@
 	(wire
 		(pts
+			(xy 459.74 182.88) (xy 459.74 181.61)
+		)
+		(stroke
+			(width 0)
+			(type default)
+		)
+	)
+	(wire
+		(pts
 			(xy 191.77 167.64) (xy 191.77 187.96)
 		)
@@
 	(wire
 		(pts
-			(xy 450.85 168.91) (xy 450.85 173.99)
-		)
-		(stroke
-			(width 0)
-			(type default)
-		)
-	)
-	(wire
-		(pts
 			(xy 473.71 119.38) (xy 485.14 119.38)
 		)
@@
 	(wire
 		(pts
-			(xy 450.85 173.99) (xy 450.85 182.88)
+			(xy 450.85 168.91) (xy 450.85 173.99)
 		)
 		(stroke
@@
 	(wire
 		(pts
+			(xy 441.96 181.61) (xy 441.96 182.88)
+		)
+		(stroke
+			(width 0)
+			(type default)
+		)
+	)
+	(wire
+		(pts
 			(xy 116.84 187.96) (xy 116.84 208.28)
 		)
@@
 	(wire
 		(pts
+			(xy 450.85 173.99) (xy 450.85 181.61)
+		)
+		(stroke
+			(width 0)
+			(type default)
+		)
+	)
+	(wire
+		(pts
 			(xy 85.09 180.34) (xy 97.79 180.34)
 		)
@@
 	(wire
 		(pts
-			(xy 449.58 182.88) (xy 450.85 182.88)
+			(xy 449.58 181.61) (xy 450.85 181.61)
 		)
 		(stroke
@@
 	(wire
 		(pts
-			(xy 450.85 182.88) (xy 452.12 182.88)
+			(xy 450.85 181.61) (xy 452.12 181.61)
 		)
 		(stroke
@@
 			)
 		)
-		(property "Footprint" "PCM_Resistor_SMD_AKL:R_0201_0603Metric"
+		(property "Footprint" "Resistor_SMD:R_0805_2012Metric"
 			(at 478.409 163.068 0)
 			(effects
@@
 			)
 		)
-		(property "Footprint" "Capacitor_SMD:C_0402_1005Metric"
+		(property "Footprint" "Capacitor_SMD:C_1206_3216Metric"
 			(at 461.3148 111.76 0)
 			(effects
@@
 			)
 		)
-		(property "Footprint" "PCM_Resistor_SMD_AKL:R_0402_1005Metric"
+		(property "Footprint" "Resistor_SMD:R_0805_2012Metric"
 			(at 388.239 133.858 0)
 			(effects
@@
 			)
 		)
-		(property "Footprint" "Capacitor_SMD:C_0402_1005Metric"
+		(property "Footprint" "Capacitor_SMD:C_1206_3216Metric"
 			(at 484.1748 111.76 0)
 			(effects
@@
 			)
 		)
-		(property "Footprint" "Capacitor_SMD:C_0201_0603Metric"
+		(property "Footprint" "Capacitor_SMD:C_1206_3216Metric"
 			(at 124.46 58.42 0)
 			(effects
@@
 			)
 		)
-		(property "Footprint" "Capacitor_SMD:C_0402_1005Metric"
+		(property "Footprint" "Capacitor_SMD:C_1206_3216Metric"
 			(at 303.53 74.93 0)
 			(effects
@@
 			)
 		)
-		(property "Footprint" "Capacitor_SMD:C_0402_1005Metric"
+		(property "Footprint" "Capacitor_SMD:C_1206_3216Metric"
 			(at 274.32 48.26 0)
 			(effects
@@
 			)
 		)
-		(property "Footprint" "Capacitor_SMD:C_0402_1005Metric"
+		(property "Footprint" "Capacitor_SMD:C_1206_3216Metric"
 			(at 341.63 74.93 0)
 			(effects
@@
 			)
 		)
-		(property "Footprint" "Capacitor_SMD:C_0402_1005Metric"
+		(property "Footprint" "Capacitor_SMD:C_1206_3216Metric"
 			(at 290.83 74.93 0)
 			(effects
@@
 			)
 		)
-		(property "Footprint" "Capacitor_SMD:C_0402_1005Metric"
+		(property "Footprint" "Capacitor_SMD:C_1206_3216Metric"
 			(at 278.13 74.93 0)
 			(effects
@@
 			)
 		)
-		(property "Footprint" "Capacitor_SMD:C_0402_1005Metric"
+		(property "Footprint" "Capacitor_SMD:C_1206_3216Metric"
 			(at 316.23 74.93 0)
 			(effects
@@
 			)
 		)
-		(property "Footprint" "PCM_Resistor_SMD_AKL:R_0402_1005Metric"
+		(property "Footprint" "Resistor_SMD:R_0402_1005Metric"
 			(at 215.392 30.099 0)
 			(effects
@@
 			)
 		)
-		(property "Footprint" "PCM_Resistor_SMD_AKL:R_0402_1005Metric"
+		(property "Footprint" "Resistor_SMD:R_0402_1005Metric"
 			(at 503.682 156.21 90)
 			(effects
@@
 			)
 		)
-		(property "Footprint" "Capacitor_SMD:C_0201_0603Metric"
+		(property "Footprint" "Capacitor_SMD:C_0805_2012Metric"
 			(at 457.2 209.8548 0)
 			(effects
@@
 			)
 		)
-		(property "Footprint" "Capacitor_SMD:C_0402_1005Metric"
+		(property "Footprint" "Capacitor_SMD:C_1206_3216Metric"
 			(at 254 74.93 0)
 			(effects
@@
 	(symbol
 		(lib_id "Device:R")
-		(at 445.77 182.88 90)
+		(at 445.77 181.61 90)
 		(unit 1)
 		(exclude_from_sim no)
@@
 		(dnp no)
 		(property "Reference" "R15"
-			(at 446.786 185.674 90)
+			(at 446.786 184.404 90)
 			(effects
 				(font
@@
 		)
 		(property "Value" "10K"
-			(at 446.786 188.214 90)
+			(at 446.786 186.944 90)
 			(effects
 				(font
@@
 			)
 		)
-		(property "Footprint" "PCM_Resistor_SMD_AKL:R_1206_3216Metric"
-			(at 445.77 184.658 90)
+		(property "Footprint" "Resistor_SMD:R_1206_3216Metric"
+			(at 445.77 183.388 90)
 			(effects
 				(font
@@
 		)
 		(property "Datasheet" "~"
-			(at 445.77 182.88 0)
+			(at 445.77 181.61 0)
 			(effects
 				(font
@@
 		)
 		(property "Description" ""
-			(at 445.77 182.88 0)
+			(at 445.77 181.61 0)
 			(effects
 				(font
@@
 			)
 		)
-		(property "Footprint" "Capacitor_SMD:C_0402_1005Metric"
+		(property "Footprint" "Capacitor_SMD:C_1206_3216Metric"
 			(at 262.89 48.26 0)
 			(effects
@@
 			)
 		)
-		(property "Footprint" "Capacitor_SMD:C_0201_0603Metric"
+		(property "Footprint" "Capacitor_SMD:C_0805_2012Metric"
 			(at 325.12 39.6748 0)
 			(effects
@@
 			)
 		)
-		(property "Footprint" "PCM_Resistor_SMD_AKL:R_0201_0603Metric"
+		(property "Footprint" "Resistor_SMD:R_0805_2012Metric"
 			(at 486.029 163.068 0)
 			(effects
@@
 			)
 		)
-		(property "Footprint" "Capacitor_SMD:C_0402_1005Metric"
+		(property "Footprint" "Capacitor_SMD:C_1206_3216Metric"
 			(at 33.02 68.58 0)
 			(effects
@@
 			)
 		)
-		(property "Footprint" "PCM_Resistor_SMD_AKL:R_0402_1005Metric"
+		(property "Footprint" "Resistor_SMD:R_0402_1005Metric"
 			(at 217.932 30.099 0)
 			(effects
@@
 			)
 		)
-		(property "Footprint" "Capacitor_SMD:C_0402_1005Metric"
+		(property "Footprint" "Capacitor_SMD:C_1206_3216Metric"
 			(at 419.4048 111.76 0)
 			(effects
@@
 			)
 		)
-		(property "Footprint" "PCM_Resistor_SMD_AKL:R_0402_1005Metric"
+		(property "Footprint" "Resistor_SMD:R_0402_1005Metric"
 			(at 322.199 178.308 0)
 			(effects
@@
 			)
 		)
-		(property "Footprint" "Capacitor_SMD:C_0402_1005Metric"
+		(property "Footprint" "Capacitor_SMD:C_1206_3216Metric"
 			(at 472.7448 111.76 0)
 			(effects
@@
 			)
 		)
-		(property "Footprint" "Capacitor_SMD:C_0402_1005Metric"
+		(property "Footprint" "Capacitor_SMD:C_1206_3216Metric"
 			(at 354.33 74.93 0)
 			(effects
@@
 			)
 		)
-		(property "Footprint" "PCM_Resistor_SMD_AKL:R_1206_3216Metric"
+		(property "Footprint" "Resistor_SMD:R_1206_3216Metric"
 			(at 267.589 171.958 0)
 			(effects
@@
 			)
 		)
-		(property "Footprint" "Capacitor_SMD:C_0402_1005Metric"
+		(property "Footprint" "Capacitor_SMD:C_1206_3216Metric"
 			(at 265.43 74.93 0)
 			(effects
@@
 	(symbol
 		(lib_id "Device:C")
-		(at 455.93 182.88 270)
+		(at 455.93 181.61 270)
 		(unit 1)
 		(exclude_from_sim no)
@@
 		(dnp no)
 		(property "Reference" "C22"
-			(at 457.708 178.816 90)
+			(at 457.708 177.546 90)
 			(effects
 				(font
@@
 		)
 		(property "Value" "100nF"
-			(at 457.708 181.356 90)
+			(at 457.708 180.086 90)
 			(effects
 				(font
@@
 			)
 		)
-		(property "Footprint" "Capacitor_SMD:C_0402_1005Metric"
-			(at 452.12 183.8452 0)
+		(property "Footprint" "Capacitor_SMD:C_1206_3216Metric"
+			(at 452.12 182.5752 0)
 			(effects
 				(font
@@
 		)
 		(property "Datasheet" "~"
-			(at 455.93 182.88 0)
+			(at 455.93 181.61 0)
 			(effects
 				(font
@@
 		)
 		(property "Description" ""
-			(at 455.93 182.88 0)
+			(at 455.93 181.61 0)
 			(effects
 				(font
@@
 			)
 		)
-		(property "Footprint" "PCM_Resistor_SMD_AKL:R_1206_3216Metric"
+		(property "Footprint" "Resistor_SMD:R_1206_3216Metric"
 			(at 267.589 174.498 0)
 			(effects
@@
 		(on_board yes)
 		(dnp no)
-		(fields_autoplaced yes)
 		(property "Reference" "#PWR042"
 			(at 441.96 179.07 0)
@@
 		)
 		(property "Value" "+5V"
-			(at 441.96 187.96 0)
+			(at 441.96 186.69 0)
 			(effects
 				(font
@@
 			)
 		)
-		(property "Footprint" "Capacitor_SMD:C_0402_1005Metric"
+		(property "Footprint" "Capacitor_SMD:C_1206_3216Metric"
 			(at 287.02 48.26 0)
 			(effects
@@
 			)
 		)
-		(property "Footprint" "Capacitor_SMD:C_0201_0603Metric"
+		(property "Footprint" "Capacitor_SMD:C_0805_2012Metric"
 			(at 325.12 52.3748 0)
 			(effects
@@
 			)
 		)
-		(property "Footprint" "Capacitor_SMD:C_0201_0603Metric"
+		(property "Footprint" "Capacitor_SMD:C_1206_3216Metric"
 			(at 106.68 58.42 0)
 			(effects
@@
 			)
 		)
-		(property "Footprint" "Capacitor_SMD:C_0402_1005Metric"
+		(property "Footprint" "Capacitor_SMD:C_1206_3216Metric"
 			(at 328.93 74.93 0)
 			(effects
@@
 			)
 		)
-		(property "Footprint" "Capacitor_SMD:C_0201_0603Metric"
+		(property "Footprint" "Capacitor_SMD:C_0805_2012Metric"
 			(at 457.2 197.1548 0)
 			(effects
@@
 			)
 		)
-		(property "Footprint" "PCM_Resistor_SMD_AKL:R_1206_3216Metric"
+		(property "Footprint" "Resistor_SMD:R_1206_3216Metric"
 			(at 494.792 156.21 90)
 			(effects
@@
 			)
 		)
-		(property "Footprint" "Capacitor_SMD:C_0402_1005Metric"
+		(property "Footprint" "Capacitor_SMD:C_1206_3216Metric"
 			(at 430.8348 111.76 0)
 			(effects
@@
 		(on_board yes)
 		(dnp no)
-		(fields_autoplaced yes)
 		(property "Reference" "#PWR043"
 			(at 459.74 189.23 0)
@@
 		)
 		(property "Value" "GND"
-			(at 459.74 187.96 0)
+			(at 459.74 186.69 0)
 			(effects
 				(font
@@
 			)
 		)
-		(property "Footprint" "PCM_Resistor_SMD_AKL:R_0402_1005Metric"
+		(property "Footprint" "Resistor_SMD:R_0805_2012Metric"
 			(at 388.239 136.398 0)
 			(effects
@@
 			)
 		)
-		(property "Footprint" "PCM_Resistor_SMD_AKL:R_0201_0603Metric"
+		(property "Footprint" "Resistor_SMD:R_0805_2012Metric"
 			(at 493.268 164.211 0)
 			(effects
@@
 			)
 		)
-		(property "Footprint" "PCM_Resistor_SMD_AKL:R_1206_3216Metric"
+		(property "Footprint" "Resistor_SMD:R_1206_3216Metric"
 			(at 62.738 65.151 0)
 			(effects

Commit message: redesigning whole board so everything is at the back except the XLR stuff :pf:
Parts:
- removed R10, R2: 220, Resistor_SMD:R_0805_2012Metric, symbol PCM_SL_Resistors:Resistor
- removed U2: NCP1117-1.5_SOT223, Package_TO_SOT_SMD:SOT-223-3_TabPin2, symbol Regulator_Linear:NCP1117-1.5_SOT223
- added U4: NCP1117-3.3_SOT223, Package_TO_SOT_SMD:SOT-223-3_TabPin2, symbol Regulator_Linear:NCP1117-3.3_SOT223
- R1: value 220 -> 680
- R13, R3, R4: footprint Resistor_SMD:R_0402_1005Metric -> Resistor_SMD:R_0805_2012Metric
Connections:
- net +3V3: now also U4.2 (VO)
- net GND: now also R1.1, U4.1 (GND)
- net VBUS: now also U4.3 (VI)
- net at GL850G1.4 (RREF): now also R1.2; no longer R1.1
Changed lines of the file:
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@@
 	(wire
 		(pts
-			(xy 488.95 170.18) (xy 488.95 168.91)
+			(xy 488.95 158.75) (xy 488.95 170.18)
 		)
 		(stroke
@@
 	(wire
 		(pts
+			(xy 481.33 158.75) (xy 488.95 158.75)
+		)
+		(stroke
+			(width 0)
+			(type default)
+		)
+	)
+	(wire
+		(pts
 			(xy 455.93 125.73) (xy 455.93 123.19)
 		)
@@
 	(wire
 		(pts
-			(xy 488.95 161.29) (xy 488.95 158.75)
-		)
-		(stroke
-			(width 0)
-			(type default)
-		)
-	)
-	(wire
-		(pts
 			(xy 68.58 229.87) (xy 68.58 208.28)
 		)
@@
 		(lib_id "PCM_SL_Resistors:Resistor")
 		(at 477.52 158.75 0)
+		(mirror y)
 		(unit 1)
 		(exclude_from_sim no)
@@
 			)
 		)
-		(property "Value" "220"
+		(property "Value" "680"
 			(at 477.52 160.782 0)
 			(effects
@@
 		)
 		(property "Footprint" "Resistor_SMD:R_0805_2012Metric"
-			(at 478.409 163.068 0)
+			(at 476.631 163.068 0)
 			(effects
 				(font
@@
 		)
 		(property "Datasheet" ""
-			(at 478.028 158.75 0)
+			(at 477.012 158.75 0)
 			(effects
 				(font
@@
 			)
 		)
-		(property "Footprint" "Resistor_SMD:R_0402_1005Metric"
+		(property "Footprint" "Resistor_SMD:R_0805_2012Metric"
 			(at 215.392 30.099 0)
 			(effects
@@
 			)
 		)
-		(property "Footprint" "Resistor_SMD:R_0402_1005Metric"
+		(property "Footprint" "Resistor_SMD:R_0805_2012Metric"
 			(at 503.682 156.21 90)
 			(effects
@@
 	)
 	(symbol
-		(lib_id "PCM_SL_Resistors:Resistor")
-		(at 485.14 158.75 0)
-		(unit 1)
-		(exclude_from_sim no)
-		(in_bom yes)
-		(on_board yes)
-		(dnp no)
-		(property "Reference" "R2"
-			(at 485.14 162.052 0)
-			(effects
-				(font
-					(size 0.762 0.762)
-				)
-			)
-		)
-		(property "Value" "220"
-			(at 485.14 160.782 0)
-			(effects
-				(font
-					(size 1.27 1.27)
-				)
-			)
-		)
-		(property "Footprint" "Resistor_SMD:R_0805_2012Metric"
-			(at 486.029 163.068 0)
-			(effects
-				(font
-					(size 1.27 1.27)
-				)
-				(hide yes)
-			)
-		)
-		(property "Datasheet" ""
-			(at 485.648 158.75 0)
-			(effects
-				(font
-					(size 1.27 1.27)
-				)
-				(hide yes)
-			)
-		)
-		(property "Description" "1/4W Resistor"
-			(at 485.14 158.75 0)
-			(effects
-				(font
-					(size 1.27 1.27)
-				)
-				(hide yes)
-			)
-		)
-		(pin "2"
-		)
-		(pin "1"
-		)
-		(instances
-			(project "Modulus"
-				(path "/b7b015a6-2592-43f0-be2e-0d1cbff8986d"
-					(reference "R2")
-					(unit 1)
-				)
-			)
-		)
-	)
-	(symbol
 		(lib_id "SCOTOKEEBS:Placeholder_Keyswitch")
 		(at 119.38 232.41 0)
@@
 			)
 		)
-		(property "Footprint" "Resistor_SMD:R_0402_1005Metric"
+		(property "Footprint" "Resistor_SMD:R_0805_2012Metric"
 			(at 217.932 30.099 0)
 			(effects
@@
 	)
 	(symbol
+		(lib_id "Regulator_Linear:NCP1117-3.3_SOT223")
+		(at 115.57 53.34 0)
+		(unit 1)
+		(exclude_from_sim no)
+		(in_bom yes)
+		(on_board yes)
+		(dnp no)
+		(fields_autoplaced yes)
+		(property "Reference" "U4"
+			(at 115.57 46.99 0)
+			(effects
+				(font
+					(size 1.27 1.27)
+				)
+			)
+		)
+		(property "Value" "NCP1117-3.3_SOT223"
+			(at 115.57 49.53 0)
+			(effects
+				(font
+					(size 1.27 1.27)
+				)
+			)
+		)
+		(property "Footprint" "Package_TO_SOT_SMD:SOT-223-3_TabPin2"
+			(at 115.57 48.26 0)
+			(effects
+				(font
+					(size 1.27 1.27)
+				)
+				(hide yes)
+			)
+		)
+		(property "Datasheet" "http://www.onsemi.com/pub_link/Collateral/NCP1117-D.PDF"
+			(at 118.11 59.69 0)
+			(effects
+				(font
+					(size 1.27 1.27)
+				)
+				(hide yes)
+			)
+		)
+		(property "Description" "1A Low drop-out regulator, Fixed Output 3.3V, SOT-223"
+			(at 115.57 53.34 0)
+			(effects
+				(font
+					(size 1.27 1.27)
+				)
+				(hide yes)
+			)
+		)
+		(pin "3"
+		)
+		(pin "1"
+		)
+		(pin "2"
+		)
+		(instances
+			(project ""
+				(path "/b7b015a6-2592-43f0-be2e-0d1cbff8986d"
+					(reference "U4")
+					(unit 1)
+				)
+			)
+		)
+	)
+	(symbol
 		(lib_id "SCOTOKEEBS:Placeholder_Keyswitch")
 		(at 181.61 170.18 0)
@@
 	)
 	(symbol
-		(lib_id "Regulator_Linear:NCP1117-1.5_SOT223")
-		(at 115.57 53.34 0)
-		(unit 1)
-		(exclude_from_sim no)
-		(in_bom yes)
-		(on_board yes)
-		(dnp no)
-		(fields_autoplaced yes)
-		(property "Reference" "U2"
-			(at 115.57 46.99 0)
-			(effects
-				(font
-					(size 1.27 1.27)
-				)
-			)
-		)
-		(property "Value" "NCP1117-1.5_SOT223"
-			(at 115.57 49.53 0)
-			(effects
-				(font
-					(size 1.27 1.27)
-				)
-			)
-		)
-		(property "Footprint" "Package_TO_SOT_SMD:SOT-223-3_TabPin2"
-			(at 115.57 48.26 0)
-			(effects
-				(font
-					(size 1.27 1.27)
-				)
-				(hide yes)
-			)
-		)
-		(property "Datasheet" "http://www.onsemi.com/pub_link/Collateral/NCP1117-D.PDF"
-			(at 118.11 59.69 0)
-			(effects
-				(font
-					(size 1.27 1.27)
-				)
-				(hide yes)
-			)
-		)
-		(property "Description" "1A Low drop-out regulator, Fixed Output 1.5V, SOT-223"
-			(at 115.57 53.34 0)
-			(effects
-				(font
-					(size 1.27 1.27)
-				)
-				(hide yes)
-			)
-		)
-		(pin "3"
-		)
-		(pin "1"
-		)
-		(pin "2"
-		)
-		(instances
-			(project ""
-				(path "/b7b015a6-2592-43f0-be2e-0d1cbff8986d"
-					(reference "U2")
-					(unit 1)
-				)
-			)
-		)
-	)
-	(symbol
 		(lib_id "SCOTOKEEBS:Placeholder_Diode")
 		(at 97.79 176.53 90)
@@
 					(unit 1)
 				)
-			)
-		)
-	)
-	(symbol
-		(lib_id "PCM_SL_Resistors:Resistor")
-		(at 488.95 165.1 90)
-		(unit 1)
-		(exclude_from_sim no)
-		(in_bom yes)
-		(on_board yes)
-		(dnp no)
-		(property "Reference" "R10"
-			(at 492.252 165.1 0)
-			(effects
-				(font
-					(size 0.762 0.762)
-				)
-			)
-		)
-		(property "Value" "220"
-			(at 490.982 165.1 0)
-			(effects
-				(font
-					(size 1.27 1.27)
-				)
-			)
-		)
-		(property "Footprint" "Resistor_SMD:R_0805_2012Metric"
-			(at 493.268 164.211 0)
-			(effects
-				(font
-					(size 1.27 1.27)
-				)
-				(hide yes)
-			)
-		)
-		(property "Datasheet" ""
-			(at 488.95 164.592 0)
-			(effects
-				(font
-					(size 1.27 1.27)
-				)
-				(hide yes)
-			)
-		)
-		(property "Description" "1/4W Resistor"
-			(at 488.95 165.1 0)
-			(effects
-				(font
-					(size 1.27 1.27)
-				)
-				(hide yes)
-			)
-		)
-		(pin "2"
-		)
-		(pin "1"
-		)
-		(instances
-			(project "Modulus"
-				(path "/b7b015a6-2592-43f0-be2e-0d1cbff8986d"
-					(reference "R10")
-					(unit 1)
-				)
