File: Modulus.kicad_sch (KiCad schematic)
At the start: 230 parts, among them J1 XLR3, J2 USB_C_Receptacle_USB2.0_16P, J3 USB_A, J4 USB_A, J5 XLR3, J6 OLED_128x32, P1 Keyswitch, Q1 Keyswitch, SW1 Push_Button, T1 Keyswitch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

Commit message: Moved everything to the back
Parts:
- D91: footprint Green_LED:0603 -> LED_THT:LED_D5.0mm
Changed lines of the file:
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@@
 			)
 		)
-		(property "Footprint" "Green_LED:0603"
+		(property "Footprint" "LED_THT:LED_D5.0mm"
 			(at 327.66 168.91 0)
 			(effects
