File: kicad/Modulus.kicad_pcb (KiCad board)
At the start: 2 copper layers, 295.6 x 183 mm, 231 parts, among them J1 XLR3, J2 USB_C_Receptacle_USB2.0_16P, J3 USB_A, J4 USB_A, J5 XLR3, J6 OLED_128x32, P1 Keyswitch, Q1 Keyswitch, SW1 Push_Button, T1 Keyswitch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

Commit message: removed lock file
Parts:
- added A1: Raspberry_Pi_Pico_THT, PCM_SL_Development_Boards:raspberry_pi_pico_THT, F.Cu at (348.1, 124.7)
- added D1: Diode, Diode_SMD:D_SMA, B.Cu at (371.0, 44.1)
- added D10: Diode, Diode_SMD:D_SMA, B.Cu at (390.1, 120.3)
- added D11: Diode, Diode_SMD:D_SMA, B.Cu at (409.1, 44.1)
- added D12: Diode, Diode_SMD:D_SMA, B.Cu at (409.1, 63.2)
- added D13: Diode, Diode_SMD:D_SMA, B.Cu at (412.1, 72.2)
- added D14: Diode, Diode_SMD:D_SMA, B.Cu at (409.1, 101.3)
- added D15: Diode, Diode_SMD:D_SMA, B.Cu at (409.1, 120.3)
- added D16: Diode, Diode_SMD:D_SMA, B.Cu at (428.2, 44.1)
- added D17: Diode, Diode_SMD:D_SMA, B.Cu at (428.2, 63.2)
- added D18: Diode, Diode_SMD:D_SMA, B.Cu at (425.2, 73.2)
- added D19: Diode, Diode_SMD:D_SMA, B.Cu at (425.2, 101.3)
- added D2: Diode, Diode_SMD:D_SMA, B.Cu at (371.0, 63.2)
- added D20: Diode, Diode_SMD:D_SMA, B.Cu at (447.2, 44.1)
- added D21: Diode, Diode_SMD:D_SMA, B.Cu at (447.2, 63.2)
- added D22: Diode, Diode_SMD:D_SMA, B.Cu at (447.2, 82.2)
- added D23: Diode, Diode_SMD:D_SMA, B.Cu at (447.2, 101.3)
- added D24: Diode, Diode_SMD:D_SMA, B.Cu at (447.2, 120.3)
- added D25: D_Generic, Diode_SMD:D_SMA, B.Cu at (331.6, 70.7)
- added D3: Diode, Diode_SMD:D_SMA, B.Cu at (371.0, 82.2)
- added D4: Diode, Diode_SMD:D_SMA, B.Cu at (371.0, 101.3)
- added D5: Diode, Diode_SMD:D_SMA, B.Cu at (371.0, 120.3)
- added D6: Diode, Diode_SMD:D_SMA, B.Cu at (390.1, 44.1)
- added D7: Diode, Diode_SMD:D_SMA, B.Cu at (390.1, 63.2)
- added D8: Diode, Diode_SMD:D_SMA, B.Cu at (390.1, 82.2)
- added D9: Diode, Diode_SMD:D_SMA, B.Cu at (390.1, 101.3)
- added J10: XLR3, NC3FAAH:NEUTRIK_NC3FAAH, F.Cu at (333.2, 29.7)
- added J9: XLR3, NC3FAAH:NEUTRIK_NC3FAAH, F.Cu at (333.2, 58.1)
- added S1: ~, PCM_Switch_Keyboard_Hotswap_Kailh:SW_Hotswap_Kailh_MX_1.00u, F.Cu at (362.0, 40.5)
- added S10: ~, PCM_Switch_Keyboard_Hotswap_Kailh:SW_Hotswap_Kailh_MX_1.00u, F.Cu at (381.1, 116.7)
- added S11: ~, PCM_Switch_Keyboard_Hotswap_Kailh:SW_Hotswap_Kailh_MX_1.00u, F.Cu at (400.1, 40.5)
- added S12: ~, PCM_Switch_Keyboard_Hotswap_Kailh:SW_Hotswap_Kailh_MX_1.00u, F.Cu at (400.1, 59.5)
- added S13: ~, PCM_Switch_Keyboard_Hotswap_Kailh:SW_Hotswap_Kailh_MX_1.00u, F.Cu at (400.1, 78.6)
- added S14: ~, PCM_Switch_Keyboard_Hotswap_Kailh:SW_Hotswap_Kailh_MX_1.00u, F.Cu at (400.1, 97.7)
- added S15: ~, PCM_Switch_Keyboard_Hotswap_Kailh:SW_Hotswap_Kailh_MX_1.00u, F.Cu at (400.1, 116.7)
- added S16: ~, PCM_Switch_Keyboard_Hotswap_Kailh:SW_Hotswap_Kailh_MX_1.00u, F.Cu at (419.2, 40.5)
- added S17: ~, PCM_Switch_Keyboard_Hotswap_Kailh:SW_Hotswap_Kailh_MX_1.00u, F.Cu at (419.2, 59.5)
- added S18: ~, PCM_Switch_Keyboard_Hotswap_Kailh:SW_Hotswap_Kailh_MX_1.50u_90deg, F.Cu at (419.2, 83.4)
- added S19: ~, PCM_Switch_Keyboard_Hotswap_Kailh:SW_Hotswap_Kailh_MX_1.50u_90deg, F.Cu at (419.2, 111.9)
- added S2: ~, PCM_Switch_Keyboard_Hotswap_Kailh:SW_Hotswap_Kailh_MX_1.00u, F.Cu at (362.0, 59.5)
- added S20: ~, PCM_Switch_Keyboard_Hotswap_Kailh:SW_Hotswap_Kailh_MX_1.00u, F.Cu at (438.2, 40.5)
- added S21: ~, PCM_Switch_Keyboard_Hotswap_Kailh:SW_Hotswap_Kailh_MX_1.00u, F.Cu at (438.2, 59.6)
- added S22: ~, PCM_Switch_Keyboard_Hotswap_Kailh:SW_Hotswap_Kailh_MX_1.00u, F.Cu at (438.2, 78.6)
- added S23: ~, PCM_Switch_Keyboard_Hotswap_Kailh:SW_Hotswap_Kailh_MX_1.00u, F.Cu at (438.2, 97.7)
- added S24: ~, PCM_Switch_Keyboard_Hotswap_Kailh:SW_Hotswap_Kailh_MX_1.00u, F.Cu at (438.2, 116.7)
- added S3: ~, PCM_Switch_Keyboard_Hotswap_Kailh:SW_Hotswap_Kailh_MX_1.00u, F.Cu at (362.0, 78.6)
- added S4: ~, PCM_Switch_Keyboard_Hotswap_Kailh:SW_Hotswap_Kailh_MX_1.00u, F.Cu at (362.0, 97.7)
- added S5: ~, PCM_Switch_Keyboard_Hotswap_Kailh:SW_Hotswap_Kailh_MX_1.00u, F.Cu at (362.0, 116.7)
- added S6: ~, PCM_Switch_Keyboard_Hotswap_Kailh:SW_Hotswap_Kailh_MX_1.00u, F.Cu at (381.1, 40.5)
- added S7: ~, PCM_Switch_Keyboard_Hotswap_Kailh:SW_Hotswap_Kailh_MX_1.00u, F.Cu at (381.1, 59.5)
- added S8: ~, PCM_Switch_Keyboard_Hotswap_Kailh:SW_Hotswap_Kailh_MX_1.00u, F.Cu at (381.1, 78.6)
- added S9: ~, PCM_Switch_Keyboard_Hotswap_Kailh:SW_Hotswap_Kailh_MX_1.00u, F.Cu at (381.1, 97.7)
Routing:
- net NUMPAD_ROW_4: track 0.00 -> 176.6 mm, vias 0 -> 9
- net NUMPAD_ROW_3: track 0.00 -> 172.1 mm, vias 0 -> 7
- net NUMPAD_ROW_2: track 0.00 -> 148.7 mm, vias 0 -> 9
- net NUMPAD_ROW_1: track 0.00 -> 129.0 mm, vias 0 -> 9
- net NUMPAD_COL_4: track 0.00 -> 127.1 mm, vias 0 -> 1
- net NUMPAD_COL_0: track 0.00 -> 124.9 mm, vias 0 -> 1
- net NUMPAD_COL_2: track 0.00 -> 115.1 mm, vias 0 -> 1
- net NUMPAD_COL_3: track 0.00 -> 113.2 mm, vias 0 -> 1
- net NUMPAD_COL_1: track 0.00 -> 111.0 mm, vias 0 -> 1
- net NUMPAD_ROW_0: track 0.00 -> 96.8 mm, vias 0 -> 1
- net NUMPAD_XLR_RX: track 0.00 -> 64.4 mm
- net NUMPAD_XLR_CSn: track 0.00 -> 56.9 mm
- net POWER: track 0.00 -> 51.9 mm
- net UNFILTERED-POWER: track 0.00 -> 46.4 mm
- net NUMPAD_XLR_SCK: track 0.00 -> 40.1 mm
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Other:
- board size 295.6 x 183 mm -> 436.2 x 183.3 mm
- board text added: "Ensure that keyboard is disconnected from power before attaching XLR modules"
- board text added: "Number + Macro Pad"
